Commit message: camera rotation can be changed in sensor_properties.xacro in selfie_desccription folder

File: src/selfie-simulator/selfie_description/urdf/selfie.xacro (robot description, xacro)
@@ -2,4 +2,5 @@
 <robot name="selfie" xmlns:xacro="http://www.ros.org/wiki/xacro">
   <xacro:include filename="$(find selfie_description)/urdf/macros.xacro" />
+  <xacro:include filename="$(find selfie_description)/urdf/selfie.gazebo" />
   <!-- Add chassis and it's inertia link -->
   <link name="base_link" />
@@ -215,10 +216,6 @@
   </link>
   <joint name="lens_joint" type="fixed">
-    <origin xyz="0 0 0.4" rpy="0 0.26 0"/>
-    <parent link="base_camera_link"/>
-    <child link="camera_link"/>
-    <axis xyz="0 0 1" />
-  </joint>
-<xacro:include filename="$(find selfie_description)/urdf/selfie.gazebo" />
+    <xacro:lens_joint_pose/>
+  </joint>
 <xacro:include filename="$(find selfie_description)/urdf/materials.xacro" />
 </robot>

File: src/selfie-simulator/selfie_description/urdf/sensor_properties.xacro (robot description, xacro)
@@ -32,3 +32,9 @@
     <distortionT2>0.0</distortionT2>
   </xacro:macro>
+  <xacro:macro name="lens_joint_pose">
+    <origin xyz="0 0 0.4" rpy="0 0.26 0"/>  <!--26-->
+    <parent link="base_camera_link"/>
+    <child link="camera_link"/>
+    <axis xyz="0 0 1" />
+  </xacro:macro>
 </robot>
