Commit message: Geometries have now correct dimensions. Only visual properties of wheels was left unchanged, so they might look stupid.

File: src/selfie-simulator/selfie_description/urdf/macros.xacro (robot description, xacro)
@@ -39,7 +39,7 @@
 <!-- geometry macros -->
 <xacro:macro name="chassis_geometry">
-  <origin xyz="0 0 0" rpy="0 0 0" />
+  <origin xyz="0.11 0 0" rpy="0 0 0" /> <!-- origin xyz="-0.08 0 0" rpy="0 0 0"-->
   <geometry>
-    <mesh filename="package://selfie_description/meshes/chassis.STL" />
+    <mesh filename="package://selfie_description/meshes/my_chasis.STL" />
   </geometry>
 </xacro:macro>
@@ -83,5 +83,5 @@
   <origin xyz="0 0 -0.0225" rpy="0 0 0" />
   <geometry>
-    <cylinder length="0.045" radius="0.05" />
+    <cylinder length="0.03" radius="0.03" />
   </geometry>
 </xacro:macro>
@@ -89,5 +89,5 @@
   <origin xyz="0 0 0.0225" rpy="0 0 0" />
   <geometry>
-    <cylinder length="0.045" radius="0.05" />  <!-- changed from 0.045   -->
+    <cylinder length="0.03" radius="0.03" />  <!-- changed from 0.045   -->
   </geometry>
 </xacro:macro>

File: src/selfie-simulator/selfie_description/urdf/selfie.xacro (robot description, xacro)
@@ -35,10 +35,10 @@
       <material name="black" />
     </visual>
-    <collision>robot
+    <collision>
       <xacro:left_wheels_collision_geometry />
     </collision>
   </link>
   <joint name="left_rear_wheel_joint" type="continuous">
-    <origin xyz="0 0.1 0" rpy="1.5708 0 0" />
+    <origin xyz="0 0.05 0" rpy="1.5708 0 0" />
     <parent link="chassis" />
     <child link="left_rear_wheel" />
@@ -61,5 +61,5 @@
   </link>
   <joint name="right_rear_wheel_joint" type="continuous">
-    <origin xyz="0 -0.1 0" rpy="1.5708 0 0" />
+    <origin xyz="0 -0.05 0" rpy="1.5708 0 0" />
     <parent link="chassis" />
     <child link="right_rear_wheel" />
@@ -79,5 +79,5 @@
   </link>
   <joint name="left_steering_hinge_joint" type="revolute">
-    <origin xyz="0.325 0.1 0" rpy="0 1.5708 0" />
+    <origin xyz="0.225 0.06 0" rpy="0 1.5708 0" /> <!-- 0.325-->
     <parent link="chassis" />
     <child link="left_steering_hinge" />
@@ -97,5 +97,5 @@
   </link>
   <joint name="right_steering_hinge_joint" type="continuous">
-    <origin xyz="0.325 -0.1 0" rpy="0 1.5708 0" />
+    <origin xyz="0.225 -0.06 0" rpy="0 1.5708 0" />  <!-- 0.325-->
     <parent link="chassis" />
     <child link="right_steering_hinge" />
@@ -154,5 +154,5 @@
       <origin xyz="0 0 0" rpy="0 0 0"/>
       <geometry>
-        <box size="0.1 0.1 0.1"/>
+        <box size="0.05 0.05 0.05"/>
       </geometry>
     </collision>
@@ -166,32 +166,31 @@
   </link>
   <joint name="hokuyo_joint" type="fixed">
-    <origin xyz="0.265 0.0 0.075" rpy="0 0 0"/>
-    <parent link="chassis" />
-    <child link="laser" />
-    <axis xyz="0 0 1" />
-  </joint>
-  <!-- zed camera -->
+    <xacro:lidar_pose/>
+  </joint>
+  <!-- camera -->
   <link name="base_camera_link">
     <inertial>
       <mass value="1e-5" />
-      <origin xyz="0 0 0.2" rpy="0 8 0"/>
+      <origin xyz="0 0 0" rpy="0 0 0"/> <!--origin xyz="0 0 0.2" rpy="0 0 0" -->
       <inertia ixx="1e-6" ixy="0" ixz="0" iyy="1e-6" iyz="0" izz="1e-6" />
     </inertial>
     <collision>
+      <origin xyz="0 0 0" rpy="0 0 0"/> <!--origin xyz="0 0 0" rpy="0 5 0"-->
+      <geometry>
+        <box size="0.05 0.04 0.030"/>
+      </geometry>
+    </collision>
+    <!--
+    <visual>
       <origin xyz="0 0 0" rpy="0 5 0"/>
       <geometry>
-        <box size="0.05 0.04 0.030"/>
-      </geometry>
-    </collision>
-    <visual>
-      <origin xyz="0 0 0" rpy="0 5 0"/>
-      <geometry>
-        <box size="0.05 0.04 0.030"/>
+        <box size="0.05 0.04 0.03"/>
       </geometry>
       <material name="red"/>
     </visual>
+  -->
   </link>
   <joint name="base_camera_joint" type="fixed">
-    <origin xyz="0 0 0.04" rpy="0 0 0"/>
+    <origin xyz="0 0 0" rpy="0 0 0"/>
     <parent link="chassis"/>
     <child link="base_camera_link"/>
@@ -204,13 +203,13 @@
     <inertial>
       <mass value="1e-5" />
-      <origin xyz="0 0 0.4" rpy="0 0.26 0"/>
+      <origin xyz="0 0 0" rpy="0 0 0"/> <!--0.26-->
       <inertia ixx="1e-6" ixy="0" ixz="0" iyy="1e-6" iyz="0" izz="1e-6" />
     </inertial>
     <visual>
-      <origin xyz="0 0 0.4" rpy="0 0.26 0"/>
-      <geometry>
-        <box size="0.05 0.02 0.05"/>
-      </geometry>
-      <material name="yellow"/>
+      <origin xyz="0 0 0" rpy="0 0 0"/><!--0.26-->
+      <geometry>
+        <box size="0.15 0.02 0.05"/>
+      </geometry>
+      <material name="blue"/>
     </visual>
   </link>

File: src/selfie-simulator/selfie_description/urdf/sensor_properties.xacro (robot description, xacro)
@@ -38,3 +38,34 @@
     <axis xyz="0 0 1" />
   </xacro:macro>
+  <xacro:macro name="lidar_pose">
+    <origin xyz="0.2 0.0 0.075" rpy="0 0 0"/>
+    <parent link="chassis" />
+    <child link="laser" />
+    <axis xyz="0 0 1" />
+  </xacro:macro>
+  <xacro:macro name="lidar_params">
+    <pose>0 0 0.0124 0 0 0</pose>
+    <visualize>false</visualize>
+    <update_rate>40</update_rate>
+    <ray>
+      <scan>
+        <horizontal>
+          <samples>720</samples>
+          <resolution>1</resolution>
+          <min_angle>-2.3561944902</min_angle>
+          <max_angle>2.3561944902</max_angle>
+        </horizontal>
+      </scan>
+      <range>
+        <min>0.1</min>
+        <max>20.0</max>
+        <resolution>0.01</resolution>
+      </range>
+      <noise>
+        <type>gaussian</type>
+        <mean>0.0</mean>
+        <stddev>0.05</stddev>
+      </noise>
+    </ray>
+  </xacro:macro>
 </robot>

Commit message: "floating selfie" BUG corrected. All dimensions are real now.

File: src/selfie-simulator/selfie_description/urdf/macros.xacro (robot description, xacro)
@@ -47,5 +47,5 @@
   <origin xyz="0 0 0" rpy="0 0 0" />
   <geometry>
-    <mesh filename="package://selfie_description/meshes/left_rear_wheel.STL" />
+    <mesh filename="package://selfie_description/meshes/selfie_left_rear_wheel.STL" />
   </geometry>
 </xacro:macro>
@@ -53,5 +53,5 @@
   <origin xyz="0 0 0" rpy="0 0 0" />
   <geometry>
-    <mesh filename="package://selfie_description/meshes/right_rear_wheel.STL" />
+    <mesh filename="package://selfie_description/meshes/selfie_right_rear_wheel.STL" />
   </geometry>
 </xacro:macro>
@@ -59,5 +59,5 @@
   <origin xyz="0 0 0" rpy="0 0 0" />
   <geometry>
-    <mesh filename="package://selfie_description/meshes/left_front_wheel.STL" />
+    <mesh filename="package://selfie_description/meshes/selfie_left_front_wheel.STL" />
   </geometry>
 </xacro:macro>
@@ -65,5 +65,5 @@
   <origin xyz="0 0 0" rpy="0 0 0" />
   <geometry>
-    <mesh filename="package://selfie_description/meshes/right_front_wheel.STL" />
+    <mesh filename="package://selfie_description/meshes/selfie_right_front_wheel.STL" />
   </geometry>
 </xacro:macro>

File: src/selfie-simulator/selfie_description/urdf/sensor_properties.xacro (robot description, xacro)
@@ -33,5 +33,5 @@
   </xacro:macro>
   <xacro:macro name="lens_joint_pose">
-    <origin xyz="0 0 0.4" rpy="0 0.26 0"/>  <!--26-->
+    <origin xyz="0 0 0.35" rpy="0 0.26 0"/>  <!--26-->
     <parent link="base_camera_link"/>
     <child link="camera_link"/>
@@ -65,5 +65,5 @@
         <type>gaussian</type>
         <mean>0.0</mean>
-        <stddev>0.05</stddev>
+        <stddev>0.01</stddev>
       </noise>
     </ray>

Commit message: seccond try to fix "floating selfie" BUG

File: src/selfie-simulator/selfie_description/urdf/macros.xacro (robot description, xacro)
@@ -83,5 +83,5 @@
   <origin xyz="0 0 -0.0225" rpy="0 0 0" />
   <geometry>
-    <cylinder length="0.03" radius="0.03" />
+    <cylinder length="0.0333" radius="0.03" />
   </geometry>
 </xacro:macro>
@@ -89,5 +89,5 @@
   <origin xyz="0 0 0.0225" rpy="0 0 0" />
   <geometry>
-    <cylinder length="0.03" radius="0.03" />  <!-- changed from 0.045   -->
+    <cylinder length="0.0333" radius="0.03" />  <!-- changed from 0.045   -->
   </geometry>
 </xacro:macro>
