Commit message: new launch file for f1tenth competition and new map

File: src/selfie-simulator/racecar_description/urdf/racecar.xacro (robot description, xacro)
@@ -198,4 +198,17 @@
     <!-- <limit lower="0.0" upper="0.0" effort="0.0" velocity="0.0" /> -->
   </joint>
+  <link name="imu_link"><!-- this needs to match the name in zed_wrapper/zed_tf.launch -->
+    <inertial>
+      <mass value="1e-5" />
+      <origin xyz="0 0 0" rpy="0 0 0"/>
+      <inertia ixx="1e-6" ixy="0" ixz="0" iyy="1e-6" iyz="0" izz="1e-6" />
+    </inertial>
+  </link>
+  <joint name="imu_joint" type="fixed">
+    <origin xyz="0 0 0" rpy="0 0 0"/>
+    <parent link="chassis"/>
+    <child link="imu_link"/>
+    <axis xyz="0 0 1" />
+  </joint>
   <!-- zed camera lenses -->
   <!-- It seems these have to have a non-zero mass to have a camera attached? -->
@@ -226,4 +239,5 @@
     <axis xyz="0 0 1" />
   </joint>
+  <!--  IMU joint -->
   <!-- Add the remaining xacros -->
   <xacro:include filename="$(find racecar_description)/urdf/racecar.gazebo" />

File: src/selfie-simulator/racecar_description/urdf/sensor_properties.xacro (robot description, xacro)
@@ -21,5 +21,5 @@
     <alwaysOn>true</alwaysOn>
     <updateRate>30</updateRate>    <!-- 30 -->
-    <cameraName>/camera/zed</cameraName>
+    <cameraName>/main_camera</cameraName>
     <imageTopicName>/image_raw</imageTopicName>
     <cameraInfoTopicName>/camera_info</cameraInfoTopicName>
