Commit message: launch simulator on one command

File: src/selfie-simulator/racecar_description/urdf/macros.xacro (robot description, xacro)
@@ -1,4 +1,4 @@
 <?xml version="1.0"?>
-<robot name="racecar" xmlns:xacro="http://www.ros.org/wiki/xacro">
+<robot name="selfie" xmlns:xacro="http://www.ros.org/wiki/xacro">
 <!-- inertial parameter macros -->
 <xacro:macro name="chassis_inertial_params">
@@ -41,5 +41,5 @@
   <origin xyz="0 0 0" rpy="0 0 0" />
   <geometry>
-    <mesh filename="package://f1_car_description/meshes/chassis.stl" />
+    <mesh filename="package://racecar_description/meshes/chassis.stl" />
   </geometry>
 </xacro:macro>
@@ -47,5 +47,5 @@
   <origin xyz="0 0 0" rpy="0 0 0" />
   <geometry>
-    <mesh filename="package://f1_car_description/meshes/left_wheel.stl" />
+    <mesh filename="package://racecar_description/meshes/left_wheel.stl" />
   </geometry>
 </xacro:macro>
@@ -53,5 +53,5 @@
   <origin xyz="0 0 0" rpy="0 0 0" />
   <geometry>
-    <mesh filename="package://f1_car_description/meshes/right_wheel.stl" />
+    <mesh filename="package://racecar_description/meshes/right_wheel.stl" />
   </geometry>
 </xacro:macro>
@@ -59,5 +59,5 @@
   <origin xyz="0 0 0" rpy="0 0 0" />
   <geometry>
-    <mesh filename="package://f1_car_description/meshes/left_wheel.stl" />
+    <mesh filename="package://racecar_description/meshes/left_wheel.stl" />
   </geometry>
 </xacro:macro>
@@ -65,5 +65,5 @@
   <origin xyz="0 0 0" rpy="0 0 0" />
   <geometry>
-    <mesh filename="package://f1_car_description/meshes/right_wheel.stl" />
+    <mesh filename="package://racecar_description/meshes/right_wheel.stl" />
   </geometry>
 </xacro:macro>
@@ -71,5 +71,5 @@
   <origin xyz="0 0 0" rpy="0 0 0" />
   <geometry>
-    <mesh filename="package://f1_car_description/meshes/hinge.stl" />
+    <mesh filename="package://racecar_description/meshes/hinge.stl" />
   </geometry>
 </xacro:macro>
@@ -77,5 +77,5 @@
   <origin xyz="0 0 0" rpy="0 0 0" />
   <geometry>
-    <mesh filename="package://f1_car_description/meshes/hinge.stl" />
+    <mesh filename="package://racecar_description/meshes/hinge.stl" />
   </geometry>
 </xacro:macro>

File: src/selfie-simulator/racecar_description/urdf/racecar.xacro (robot description, xacro)
@@ -1,5 +1,5 @@
 <?xml version="1.0"?>
-<robot name="racecar" xmlns:xacro="http://www.ros.org/wiki/xacro">
-  <xacro:include filename="$(find f1_car_description)/urdf/macros.xacro" />
+<robot name="selfie" xmlns:xacro="http://www.ros.org/wiki/xacro">
+  <xacro:include filename="$(find racecar_description)/urdf/macros.xacro" />
   <!-- Add chassis and it's inertia link -->
   <link name="base_link"/>

Commit message: update selfie description

File: src/selfie-simulator/racecar_description/urdf/macros.xacro (robot description, xacro)
@@ -1,4 +1,10 @@
 <?xml version="1.0"?>
 <robot name="selfie" xmlns:xacro="http://www.ros.org/wiki/xacro">
+<xacro:property name="wheel_radius" value="0.055" />
+<xacro:property name="wheel_lenght" value="0.045" />
+<!-- chassis to nadwzoize ktore dla uproszczenia uznaje za prostopadloscian -->
+<xacro:property name="chassis_x" value="0.33" />
+<xacro:property name="chassis_y" value="0.2" />
+<xacro:property name="chassis_z" value="0.1" />
 <!-- inertial parameter macros -->
 <xacro:macro name="chassis_inertial_params">
@@ -41,5 +47,5 @@
   <origin xyz="0 0 0" rpy="0 0 0" />
   <geometry>
-    <mesh filename="package://racecar_description/meshes/chassis.stl" />
+    <box size="${chassis_x} ${chassis_y} ${chassis_z}"/>
   </geometry>
 </xacro:macro>
@@ -47,5 +53,5 @@
   <origin xyz="0 0 0" rpy="0 0 0" />
   <geometry>
-    <mesh filename="package://racecar_description/meshes/left_wheel.stl" />
+    <cylinder radius="${wheel_radius}" length="${wheel_lenght}"/>
   </geometry>
 </xacro:macro>
@@ -53,5 +59,5 @@
   <origin xyz="0 0 0" rpy="0 0 0" />
   <geometry>
-    <mesh filename="package://racecar_description/meshes/right_wheel.stl" />
+    <cylinder radius="${wheel_radius}" length="${wheel_lenght}"/>
   </geometry>
 </xacro:macro>
@@ -59,5 +65,5 @@
   <origin xyz="0 0 0" rpy="0 0 0" />
   <geometry>
-    <mesh filename="package://racecar_description/meshes/left_wheel.stl" />
+    <cylinder radius="${wheel_radius}" length="${wheel_lenght}"/>
   </geometry>
 </xacro:macro>
@@ -65,5 +71,5 @@
   <origin xyz="0 0 0" rpy="0 0 0" />
   <geometry>
-    <mesh filename="package://racecar_description/meshes/right_wheel.stl" />
+    <cylinder radius="${wheel_radius}" length="${wheel_lenght}"/>
   </geometry>
 </xacro:macro>
@@ -83,5 +89,5 @@
   <origin xyz="0 0 -0.0225" rpy="0 0 0" />
   <geometry>
-    <cylinder length="0.045" radius="0.05" />
+    <cylinder radius="${wheel_radius}" length="${wheel_lenght}"/>
   </geometry>
 </xacro:macro>
@@ -89,5 +95,11 @@
   <origin xyz="0 0 0.0225" rpy="0 0 0" />
   <geometry>
-    <cylinder length="0.045" radius="0.05" />
+    <cylinder radius="${wheel_radius}" length="${wheel_lenght}"/>
+  </geometry>
+</xacro:macro>
+<xacro:macro name="lidars_main_plate">
+  <origin xyz="0 0 0" rpy="0 0 0" />
+  <geometry>
+    <mesh filename="package://racecar_description/meshes/lidars_main_plate.stl" />
   </geometry>
 </xacro:macro>

File: src/selfie-simulator/racecar_description/urdf/racecar.xacro (robot description, xacro)
@@ -3,5 +3,5 @@
   <xacro:include filename="$(find racecar_description)/urdf/macros.xacro" />
   <!-- Add chassis and it's inertia link -->
-  <link name="base_link"/>
+  <link name="base_link"/> <!-- base_link najduje sie na srodku tylnej osi -->
   <link name="chassis">
     <visual>
@@ -11,5 +11,5 @@
   </link>
   <joint name="base_link_joint" type="fixed">
-    <origin xyz="0 0 0.05" rpy="0 0 0" />
+    <origin xyz="0.165 0 0.05" rpy="0 0 0" /> <!-- 0.05 to wysokosc od ziemii -->
     <parent link="base_link" />
     <child link="chassis" />
@@ -39,6 +39,6 @@
   </link>
   <joint name="left_rear_wheel_joint" type="continuous">
-    <origin xyz="0 0.1 0" rpy="1.5708 0 0" />
-    <parent link="chassis" />
+    <origin xyz="0 0.13 0" rpy="1.5708 0 0" />
+    <parent link="base_link" />
     <child link="left_rear_wheel" />
     <axis xyz="0 0 -1" />
@@ -60,6 +60,6 @@
   </link>
   <joint name="right_rear_wheel_joint" type="continuous">
-    <origin xyz="0 -0.1 0" rpy="1.5708 0 0" />
-    <parent link="chassis" />
+    <origin xyz="0 -0.13 0" rpy="1.5708 0 0" />
+    <parent link="base_link" />
     <child link="right_rear_wheel" />
     <axis xyz="0 0 -1" />
@@ -78,6 +78,6 @@
   </link>
   <joint name="left_steering_hinge_joint" type="revolute">
-    <origin xyz="0.325 0.1 0" rpy="0 1.5708 0" />
-    <parent link="chassis" />
+    <origin xyz="0.33 0.13 0" rpy="0 1.5708 0" />
+    <parent link="base_link" />
     <child link="left_steering_hinge" />
     <axis xyz="-1 0 0" />
@@ -96,6 +96,6 @@
   </link>
   <joint name="right_steering_hinge_joint" type="continuous">
-    <origin xyz="0.325 -0.1 0" rpy="0 1.5708 0" />
-    <parent link="chassis" />
+    <origin xyz="0.33 -0.13 0" rpy="0 1.5708 0" />
+    <parent link="base_link" />
     <child link="right_steering_hinge" />
     <axis xyz="-1 0 0" />
@@ -146,5 +146,5 @@
   <xacro:wheel_transmission name="right_front_wheel" />
   <!-- Add Hokuyo laser scanner -->
-  <link name="laser">
+  <link name="left_laser">
     <inertial>
       <xacro:hokuyo_inertial_params />
@@ -164,8 +164,32 @@
     </visual>
   </link>
-  <joint name="hokuyo_joint" type="fixed">
-    <origin xyz="0.265 0.0 0.075" rpy="0 0 0"/>
-    <parent link="chassis" />
-    <child link="laser" />
+  <joint name="left_hokuyo_joint" type="fixed">
+    <origin xyz="0.01 0.1275 0.165" rpy="0 0 1.5708"/> <!-- x do przodu, z do gory -->
+    <parent link="base_link" />
+    <child link="left_laser" />
+    <axis xyz="0 0 1" />
+  </joint>
+  <link name="right_laser">
+    <inertial>
+      <xacro:hokuyo_inertial_params />
+    </inertial>
+    <collision>
+      <origin xyz="0 0 0" rpy="0 0 0"/>
+      <geometry>
+        <box size="0.1 0.1 0.1"/>
+      </geometry>
+    </collision>
+    <visual>
+      <origin xyz="0 0 0" rpy="0 0 0"/>
+      <geometry>
+        <mesh filename="package://racecar_description/meshes/hokuyo.stl"/>
+        <material name="grey" />
+      </geometry>
+    </visual>
+  </link>
+  <joint name="right_hokuyo_joint" type="fixed">
+    <origin xyz="0.01 -0.1275 0.165" rpy="0 0 -1.5708"/>
+    <parent link="base_link" />
+    <child link="right_laser" />
     <axis xyz="0 0 1" />
   </joint>
@@ -192,6 +216,6 @@
   </link>
   <joint name="zed_camera_joint" type="fixed">
-    <origin xyz="0.390 0 0.04" rpy="0 0 0"/>
-    <parent link="chassis"/>
+    <origin xyz="0.33 0 0.04" rpy="0 0 0"/>
+    <parent link="base_link"/>
     <child link="zed_camera_link"/>
     <axis xyz="0 0 1" />
@@ -207,5 +231,5 @@
   <joint name="imu_joint" type="fixed">
     <origin xyz="0 0 0" rpy="0 0 0"/>
-    <parent link="chassis"/>
+    <parent link="base_link"/>
     <child link="imu_link"/>
     <axis xyz="0 0 1" />

File: src/selfie-simulator/racecar_description/urdf/sensor_properties.xacro (robot description, xacro)
@@ -41,5 +41,5 @@
     <origin xyz="0.2 0.0 0.075" rpy="0 0 0"/>
     <parent link="chassis" />
-    <child link="laser" />
+    <child link="left_laser" />
     <axis xyz="0 0 1" />
   </xacro:macro>
